File: src/Tag/PCB/Tag PCB V1.sch (EAGLE design)
At the start: 5 parts, among them IC1 ATMEGA328P-AU, Q1 16MHz

Commit message: PCB JLC tag added
Parts:
- added 5V-IN, BAT+, BAT-: (no value), wirepad:2,15/1,0
- added C3: 100nF, rcl:C-EUC0805
- added C4: 100uF, rcl:CPOL-EUE3.5-8
- added C5: 10uF, rcl:CPOL-EUE2.5-7
- added GND-IN: GND_IN, wirepad:2,15/1,0
- added H1, H2, H3, H4: MOUNT-HOLE3.0, holes:MOUNT-HOLE3.0
- added J1: AVR_SPI_PROG_3X2PTH, SparkFun-Connectors:AVR_SPI_PROG_3X2PTH
- added R1, R2: 10k, rcl:R-EU_R0805
- added S1: RESET, SparkFun-Switches:MOMENTARY-SWITCH-SPST-PTH-6.0MM
- added U$2: UART-6PIN, Eigen Library:UART-6PIN
- added U$3: DC-DC-STEP-DOWN-LM2596, 1484249208697-powermodules:DC-DC-STEP-DOWN-LM2596
- added U$4: 18650-CHARGE-5V-OUT, Eigen Library:18650-CHARGE-5V-OUT
- Q1: value 16MHz -> 8MHz
Connections:
- new net 5V: 5V-IN.P, U$3.IN+
- new net CS: IC1.PB2_[PCINT2], U$1.CS
- new net DTR: C3.1, U$2.DTR
- new net DW-RST: IC1.PB1_[PCINT1], U$1.RST
- new net GND: C1.2, C2.2, GND-IN.P, IC1.GND_1, IC1.GND_2, IC1.GND_3, J1.6, R2.1, S1.1, U$1.GND, U$2.GND, U$3.IN-, U$3.OUT-
- new net IRQ: IC1.PD2_[PCINT18], R2.2, U$1.IRQ
- new net MISO: IC1.PB4_[PCINT4], J1.1, U$1.MISO
- new net MOSI: IC1.PB3_[PCINT3], J1.4, U$1.MOSI
- new net N$1: BAT-.P, C4.+, C5.+, U$4.B-
- new net N$2: BAT+.P, C4.-, C5.-, U$4.B+
- new net N$5: C2.1, IC1.PB7_[PCINT7], Q1.2
- new net N$6: C1.1, IC1.PB6_[PCINT6], Q1.1
- new net RST: C3.2, IC1.PC6_[RESET/PCINT14], J1.5, R1.1, S1.2
- new net RX: IC1.PD0_[PCINT16], U$2.TXD
- new net SCK: IC1.PB5_[PCINT5], J1.3, U$1.CLK
- new net TX: IC1.PD1_[PCINT17], U$2.RXD
- new net VCC: IC1.AVCC, IC1.VCC_1, IC1.VCC_2, R1.2, U$1.VCC, U$3.OUT+
Other:
- note added: "CHARGE-BOARD"
- moved on the sheet: C1, C2, Q1
