File: src/Anchor/PCB/Anchor PCB V2.brd (EAGLE design)
At the start: 95.2 x 63.2 mm, 60 parts, among them IC3 ENC28J60-I_SS, J1 SI-50154-F, J2 ISP PROG 1, J3 ISP PROG 2, J4 POWER_JACK, Y1 8MHz, Y2 8MHz, Y3 25MHz

Commit message: Removed some unnecessary resistors in Anchor V2
Parts:
- removed R14, R15, R16: 330, rcl:R0805
Connections:
- removed net N$16: R14.2, U$2.CLK
- removed net N$17: R15.2, U$2.MISO
- removed net N$18: R16.2, U$2.MOSI
- net MISO2: now also U$2.MISO; no longer R15.1
- net MOSI2: now also U$2.MOSI; no longer R16.1
- net SCK2: now also U$2.CLK; no longer R14.1
Routing:
- net SCK2: track 20.0 -> 45.8 mm
- net N$16: track 19.0 -> 0.00 mm
- net MISO2: track 19.1 -> 35.6 mm
- net N$17: track 12.8 -> 0.00 mm
- net MOSI2: track 26.3 -> 36.2 mm
- net RX1: track 42.0 -> 48.9 mm
- net N$18: track 6.70 -> 0.00 mm
- net TX1: track 36.9 -> 43.6 mm
- net RX3: track 80.7 -> 86.8 mm
- net N$3: track 20.9 -> 25.8 mm
- net RST1: track 84.3 -> 88.5 mm
- net MISO1: track 66.2 -> 62.2 mm, vias 4 -> 3
- net N$12: track 40.2 -> 43.2 mm
- net N$9: track 24.3 -> 27.2 mm
- net RST2: track 49.7 -> 52.0 mm, vias 2 -> 1
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Other:
- board size 95.2 x 63.2 mm -> 105.4 x 63.2 mm
- board text added: "5V-40V DC"
- board text added: "UART 1"
- board text added: "UART 2"

Commit message: PCB JLC tag added
Routing:
- net CS1: track 29.2 -> 24.1 mm
- net N$14: track 6.80 -> 9.15 mm
- net RST1: track 88.5 -> 90.8 mm
- net MISO1: track 62.2 -> 64.0 mm, vias 3 -> 2
- net N$11: track 4.84 -> 6.63 mm
- net N$15: track 9.83 -> 11.5 mm
- net RX3: track 86.8 -> 85.7 mm
- net TPIN+: track 51.9 -> 50.9 mm
- net GND: track 417.6 -> 417.1 mm
Other:
- board size 105.4 x 63.2 mm -> 95.2 x 63.2 mm

Commit message: Deleted CTS pin
Connections:
- removed net N$19: UART1.CTS
Changed lines of the file:
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@@
 <wire x1="78.486" y1="52.451" x2="78.89875" y2="52.86375" width="0.508" layer="1"/>
-</signal>
-<signal name="N$19">
-<contactref element="UART1" pad="CTS"/>
 </signal>
 <signal name="DTR2">
